Commit message: rotate test and speed test with new urdf

File: same_leg_urdf/10_degree.urdf (robot description, URDF)
Before this commit: robot 10_degree, 5 links, 4 joints
Joints:
- joint left_back_leg: axis 0 -0.17365 -0.98481 -> 0 0 -1; origin xyz=-0.14789 0.10144 0 rpy=1.5708 1.5708 0 -> xyz=-0.14789 0.10144 0 rpy=1.3963 1.5708 0
- joint left_front_leg: axis 0 0.17365 -0.98481 -> 0 0 -1; origin xyz=0.14789 0.10144 0 rpy=1.5708 1.5708 0 -> xyz=0.14789 0.10144 0 rpy=1.7453 1.5708 0
- joint right_front_leg: axis 0 0.17365 0.98481 -> 0 0 1; origin xyz=0.14789 -0.10144 0 rpy=1.5708 1.5708 0 -> xyz=0.14789 -0.10144 0 rpy=1.3963 1.5708 0

File: same_leg_urdf/12_degree.urdf (robot description, URDF)
Before this commit: robot 12_degree, 5 links, 4 joints
Joints:
- joint left_back_leg: axis 0 -0.20791 -0.97815 -> 0 0 -1; origin xyz=-0.15141 0.10075 0 rpy=1.5708 1.5708 0 -> xyz=-0.15141 0.10075 0 rpy=1.3614 1.5708 0
- joint left_front_leg: axis 0 0.20791 -0.97815 -> 0 0 -1; origin xyz=0.15141 0.10075 0 rpy=1.5708 1.5708 0 -> xyz=0.15141 0.10075 0 rpy=1.7802 1.5708 0
- joint right_front_leg: axis 0 0.20791 0.97815 -> 0 0 1; origin xyz=0.15141 -0.10075 0 rpy=1.5708 1.5708 0 -> xyz=0.15141 -0.10075 0 rpy=1.3614 1.5708 0

File: same_leg_urdf/14_degree.urdf (robot description, URDF)
Before this commit: robot 14_degree, 5 links, 4 joints
Joints:
- joint left_back_leg: axis 0 -0.24192 -0.9703 -> 0 0 -1; origin xyz=-0.15492 0.09994 0 rpy=1.5708 1.5708 0 -> xyz=-0.15492 0.09994 0 rpy=1.3265 1.5708 0
- joint left_front_leg: axis 0 0.24192 -0.9703 -> 0 0 -1; origin xyz=0.15492 0.09994 0 rpy=1.5708 1.5708 0 -> xyz=0.15492 0.09994 0 rpy=1.8151 1.5708 0
- joint right_front_leg: axis 0 0.24192 0.9703 -> 0 0 1; origin xyz=0.15492 -0.09994 0 rpy=1.5708 1.5708 0 -> xyz=0.15492 -0.09994 0 rpy=1.3265 1.5708 0

File: same_leg_urdf/16_degree.urdf (robot description, URDF)
Before this commit: robot 16_degree, 5 links, 4 joints
Joints:
- joint left_back_leg: axis 0 -0.27564 -0.96126 -> 0 0 -1; origin xyz=-0.15839 0.09901 0 rpy=1.5708 1.5708 0 -> xyz=-0.15839 0.09901 0 rpy=1.2915 1.5708 0
- joint left_front_leg: axis 0 0.27564 -0.96126 -> 0 0 -1; origin xyz=0.15839 0.09901 0 rpy=1.5708 1.5708 0 -> xyz=0.15839 0.09901 0 rpy=1.85 1.5708 0
- joint right_front_leg: axis 0 0.27564 0.96126 -> 0 0 1; origin xyz=0.15839 -0.09901 0 rpy=1.5708 1.5708 0 -> xyz=0.15839 -0.09901 0 rpy=1.2915 1.5708 0

File: same_leg_urdf/18_degree.urdf (robot description, URDF)
Before this commit: robot 18_degree, 5 links, 4 joints
Joints:
- joint left_back_leg: axis 0 -0.30902 -0.95106 -> 0 0 -1; origin xyz=-0.16183 0.097959 0 rpy=1.5708 1.5708 0 -> xyz=-0.16183 0.097959 0 rpy=1.2566 1.5708 0
- joint left_front_leg: axis 0 0.30902 -0.95106 -> 0 0 -1; origin xyz=0.16183 0.097959 0 rpy=1.5708 1.5708 0 -> xyz=0.16183 0.097959 0 rpy=1.885 1.5708 0
- joint right_back_leg: origin xyz=-0.16183 -0.097959 0 rpy=0.31416 1.5708 -1.5708 -> xyz=-0.16183 -0.097959 0 rpy=1.885 1.5708 0
- joint right_front_leg: axis 0 0.30902 0.95106 -> 0 0 1; origin xyz=0.16183 -0.097959 0 rpy=1.5708 1.5708 0 -> xyz=0.16183 -0.097959 0 rpy=1.2566 1.5708 0

File: same_leg_urdf/20_degree.urdf (robot description, URDF)
Before this commit: robot 20_degree, 5 links, 4 joints
Joints:
- joint left_back_leg: axis 0 -0.34202 -0.93969 -> 0 0 -1; origin xyz=-0.16523 0.096788 0 rpy=1.5708 1.5708 0 -> xyz=-0.16523 0.096788 0 rpy=1.2217 1.5708 0
- joint left_front_leg: axis 0 0.34202 -0.93969 -> 0 0 -1; origin xyz=0.16523 0.096788 0 rpy=1.5708 1.5708 0 -> xyz=0.16523 0.096788 0 rpy=1.9199 1.5708 0
- joint right_back_leg: origin xyz=-0.16523 -0.096788 0 rpy=0.34907 1.5708 -1.5708 -> xyz=-0.16523 -0.096788 0 rpy=1.9199 1.5708 0
- joint right_front_leg: axis 0 0.34202 0.93969 -> 0 0 1; origin xyz=0.16523 -0.096788 0 rpy=1.5708 1.5708 0 -> xyz=0.16523 -0.096788 0 rpy=1.2217 1.5708 0

File: same_leg_urdf/22_degree.urdf (robot description, URDF)
Before this commit: robot 22_degree, 5 links, 4 joints
Joints:
- joint left_back_leg: axis 0 -0.37461 -0.92718 -> 0 0 -1; origin xyz=-0.16858 0.0955 0 rpy=1.5708 1.5708 0 -> xyz=-0.16858 0.0955 0 rpy=1.1868 1.5708 0
- joint left_front_leg: axis 0 0.37461 -0.92718 -> 0 0 -1; origin xyz=0.16858 0.0955 0 rpy=1.5708 1.5708 0 -> xyz=0.16858 0.0955 0 rpy=1.9548 1.5708 0
- joint right_back_leg: origin xyz=-0.16858 -0.0955 0 rpy=0.38397 1.5708 -1.5708 -> xyz=-0.16858 -0.0955 0 rpy=1.9548 1.5708 0
- joint right_front_leg: axis 0 0.37461 0.92718 -> 0 0 1; origin xyz=0.16858 -0.0955 0 rpy=1.5708 1.5708 0 -> xyz=0.16858 -0.0955 0 rpy=1.1868 1.5708 0

File: same_leg_urdf/24_degree.urdf (robot description, URDF)
Before this commit: robot 24_degree, 5 links, 4 joints
Joints:
- joint left_back_leg: axis 0 -0.40674 -0.91355 -> 0 0 -1; origin xyz=-0.17189 0.094095 0 rpy=1.5708 1.5708 0 -> xyz=-0.17189 0.094095 0 rpy=1.1519 1.5708 0
- joint left_front_leg: axis 0 0.40674 -0.91355 -> 0 0 -1; origin xyz=0.17189 0.094095 0 rpy=1.5708 1.5708 0 -> xyz=0.17189 0.094095 0 rpy=1.9897 1.5708 0
- joint right_back_leg: origin xyz=-0.17189 -0.094095 0 rpy=0.41888 1.5708 -1.5708 -> xyz=-0.17189 -0.094095 0 rpy=1.9897 1.5708 0
- joint right_front_leg: axis 0 0.40674 0.91355 -> 0 0 1; origin xyz=0.17189 -0.094095 0 rpy=1.5708 1.5708 0 -> xyz=0.17189 -0.094095 0 rpy=1.1519 1.5708 0

File: same_leg_urdf/26_degree.urdf (robot description, URDF)
Before this commit: robot 26_degree, 5 links, 4 joints
Joints:
- joint left_back_leg: axis 0 -0.43837 -0.89879 -> 0 0 -1; origin xyz=-0.17515 0.092576 0 rpy=1.5708 1.5708 0 -> xyz=-0.17515 0.092576 0 rpy=1.117 1.5708 0
- joint left_front_leg: axis 0 0.43837 -0.89879 -> 0 0 -1; origin xyz=0.17515 0.092576 0 rpy=1.5708 1.5708 0 -> xyz=0.17515 0.092576 0 rpy=2.0246 1.5708 0
- joint right_front_leg: axis 0 0.43837 0.89879 -> 0 0 1; origin xyz=0.17515 -0.092576 0 rpy=1.5708 1.5708 0 -> xyz=0.17515 -0.092576 0 rpy=1.117 1.5708 0

File: same_leg_urdf/28_degree.urdf (robot description, URDF)
Before this commit: robot 28_degree, 5 links, 4 joints
Joints:
- joint left_back_leg: axis 0 -0.46947 -0.88295 -> 0 0 -1; origin xyz=-0.17836 0.090944 0 rpy=1.5708 1.5708 0 -> xyz=-0.17836 0.090944 0 rpy=1.0821 1.5708 0
- joint left_front_leg: axis 0 0.46947 -0.88295 -> 0 0 -1; origin xyz=0.17836 0.090944 0 rpy=1.5708 1.5708 0 -> xyz=0.17836 0.090944 0 rpy=2.0595 1.5708 0
- joint right_front_leg: axis 0 0.46947 0.88295 -> 0 0 1; origin xyz=0.17836 -0.090944 0 rpy=1.5708 1.5708 0 -> xyz=0.17836 -0.090944 0 rpy=1.0821 1.5708 0

File: same_leg_urdf/2_degree.urdf (robot description, URDF)
Before this commit: robot 2_degree, 5 links, 4 joints
Joints:
- joint left_back_leg: axis 0 -0.034899 -0.99939 -> 0 0 -1; origin xyz=-0.13359 0.10294 0 rpy=1.5708 1.5708 0 -> xyz=-0.13359 0.10294 0 rpy=1.5359 1.5708 0
- joint left_front_leg: axis 0 0.034899 -0.99939 -> 0 0 -1; origin xyz=0.13359 0.10294 0 rpy=1.5708 1.5708 0 -> xyz=0.13359 0.10294 0 rpy=1.6057 1.5708 0
- joint right_back_leg: origin xyz=-0.13359 -0.10294 0 rpy=0.034907 1.5708 -1.5708 -> xyz=-0.13359 -0.10294 0 rpy=1.6057 1.5708 0
- joint right_front_leg: axis 0 0.034899 0.99939 -> 0 0 1; origin xyz=0.13359 -0.10294 0 rpy=1.5708 1.5708 0 -> xyz=0.13359 -0.10294 0 rpy=1.5359 1.5708 0

File: same_leg_urdf/30_degree/urdf/30_degree.urdf (robot description, URDF)
Before this commit: robot 30_degree, 5 links, 4 joints
Joints:
- joint left_back_leg: axis 0 -0.5 -0.86603 -> 0 0 -1; origin xyz=-0.1815 0.089201 0 rpy=1.5708 1.5708 0 -> xyz=-0.1815 0.089201 0 rpy=1.0472 1.5708 0
- joint left_front_leg: axis 0 0.5 -0.86603 -> 0 0 -1; origin xyz=0.1815 0.089201 0 rpy=1.5708 1.5708 0 -> xyz=0.1815 0.089201 0 rpy=2.0944 1.5708 0
- joint right_front_leg: axis 0 0.5 0.86603 -> 0 0 1; origin xyz=0.1815 -0.089201 0 rpy=1.5708 1.5708 0 -> xyz=0.1815 -0.089201 0 rpy=1.0472 1.5708 0

File: same_leg_urdf/4_degree.urdf (robot description, URDF)
Before this commit: robot 4_degree, 5 links, 4 joints
Joints:
- joint left_back_leg: axis 0 -0.069756 -0.99756 -> 0 0 -1; origin xyz=-0.13718 0.10275 0 rpy=1.5708 1.5708 0 -> xyz=-0.13718 0.10275 0 rpy=1.501 1.5708 0
- joint left_front_leg: axis 0 0.069756 -0.99756 -> 0 0 -1; origin xyz=0.13718 0.10275 0 rpy=1.5708 1.5708 0 -> xyz=0.13718 0.10275 0 rpy=1.6406 1.5708 0
- joint right_front_leg: axis 0 0.069756 0.99756 -> 0 0 1; origin xyz=0.13718 -0.10275 0 rpy=1.5708 1.5708 0 -> xyz=0.13718 -0.10275 0 rpy=1.501 1.5708 0

File: same_leg_urdf/6_degree.urdf (robot description, URDF)
Before this commit: robot 6_degree, 5 links, 4 joints
Joints:
- joint left_back_leg: axis 0 -0.10453 -0.99452 -> 0 0 -1; origin xyz=-0.14077 0.10244 0 rpy=1.5708 1.5708 0 -> xyz=-0.14077 0.10244 0 rpy=1.4661 1.5708 0
- joint left_front_leg: axis 0 0.10453 -0.99452 -> 0 0 -1; origin xyz=0.14077 0.10244 0 rpy=1.5708 1.5708 0 -> xyz=0.14077 0.10244 0 rpy=1.6755 1.5708 0
- joint right_front_leg: axis 0 0.10453 0.99452 -> 0 0 1; origin xyz=0.14077 -0.10244 0 rpy=1.5708 1.5708 0 -> xyz=0.14077 -0.10244 0 rpy=1.4661 1.5708 0

File: same_leg_urdf/8_degree.urdf (robot description, URDF)
Before this commit: robot 8_degree, 5 links, 4 joints
Links:
- link base_link: mass 2.942 -> 2.924
Joints:
- joint left_back_leg: axis 0 -0.13917 -0.99027 -> 0 0 -1; origin xyz=-0.14433 0.102 0 rpy=1.5708 1.5708 0 -> xyz=-0.14433 0.102 0 rpy=1.4312 1.5708 0
- joint left_front_leg: axis 0 0.13917 -0.99027 -> 0 0 -1; origin xyz=0.14433 0.102 0 rpy=1.5708 1.5708 0 -> xyz=0.14433 0.102 0 rpy=1.7104 1.5708 0
- joint right_front_leg: axis 0 0.13917 0.99027 -> 0 0 1; origin xyz=0.14433 -0.102 0 rpy=1.5708 1.5708 0 -> xyz=0.14433 -0.102 0 rpy=1.4312 1.5708 0
