Commit message: env update

File: FlexipodBulletEnv/urdf/robot.urdf (robot description, URDF)
Before this commit: robot robot, 33 links, 32 joints
Links:
- removed link lb_hip_board
- removed link lb_hip_motor
- removed link lb_shank_board
- removed link lb_shank_motor
- removed link lb_thigh_motor
- removed link lf_hip_board
- removed link lf_hip_motor
- removed link lf_shank_board
- removed link lf_shank_motor
- removed link lf_thigh_motor
- removed link rb_hip_board
- removed link rb_hip_motor
- removed link rb_shank_board
- removed link rb_shank_motor
- removed link rb_thigh_motor
- removed link rf_hip_board
- removed link rf_hip_motor
- removed link rf_shank_board
- removed link rf_shank_motor
- removed link rf_thigh_motor
- added link lb_m1, mass 0.03257455734158853; collision mesh filename=mesh/lb_m1.obj; visual mesh filename=mesh/lb_m1.obj
- added link lb_m2, mass 0.03257455734158853; collision mesh filename=mesh/lb_m2.obj; visual mesh filename=mesh/lb_m2.obj
- added link lb_m3, mass 0.03257455734158853; collision mesh filename=mesh/lb_m3.obj; visual mesh filename=mesh/lb_m3.obj
- added link lb_sc, mass 0.004450137728878035; collision mesh filename=mesh/lb_sc.obj; visual mesh filename=mesh/lb_sc.obj
- added link lb_tc, mass 0.005815865339497284; collision mesh filename=mesh/lb_tc.obj; visual mesh filename=mesh/lb_tc.obj
- added link lf_m1, mass 0.03257455734158853; collision mesh filename=mesh/lf_m1.obj; visual mesh filename=mesh/lf_m1.obj
- added link lf_m2, mass 0.03257455734158853; collision mesh filename=mesh/lf_m2.obj; visual mesh filename=mesh/lf_m2.obj
- added link lf_m3, mass 0.03257455734158853; collision mesh filename=mesh/lf_m3.obj; visual mesh filename=mesh/lf_m3.obj
- added link lf_sc, mass 0.004450137728878035; collision mesh filename=mesh/lf_sc.obj; visual mesh filename=mesh/lf_sc.obj
- added link lf_tc, mass 0.005815865339497284; collision mesh filename=mesh/lf_tc.obj; visual mesh filename=mesh/lf_tc.obj
- added link rb_m1, mass 0.03257455734158853; collision mesh filename=mesh/rb_m1.obj; visual mesh filename=mesh/rb_m1.obj
- added link rb_m2, mass 0.03257455734158853; collision mesh filename=mesh/rb_m2.obj; visual mesh filename=mesh/rb_m2.obj
- added link rb_m3, mass 0.03257455734158853; collision mesh filename=mesh/rb_m3.obj; visual mesh filename=mesh/rb_m3.obj
- added link rb_sc, mass 0.004450137728878035; collision mesh filename=mesh/rb_sc.obj; visual mesh filename=mesh/rb_sc.obj
- added link rb_tc, mass 0.005815865339497284; collision mesh filename=mesh/rb_tc.obj; visual mesh filename=mesh/rb_tc.obj
- added link rf_m1, mass 0.03257455734158853; collision mesh filename=mesh/rf_m1.obj; visual mesh filename=mesh/rf_m1.obj
- added link rf_m2, mass 0.03257455734158853; collision mesh filename=mesh/rf_m2.obj; visual mesh filename=mesh/rf_m2.obj
- added link rf_m3, mass 0.03257455734158853; collision mesh filename=mesh/rf_m3.obj; visual mesh filename=mesh/rf_m3.obj
- added link rf_sc, mass 0.004450137728878035; collision mesh filename=mesh/rf_sc.obj; visual mesh filename=mesh/rf_sc.obj
- added link rf_tc, mass 0.005815865339497284; collision mesh filename=mesh/rf_tc.obj; visual mesh filename=mesh/rf_tc.obj
- link body: mass 1.0196898000000187 -> 0.376970596380699
- link lb_hip: mass 0.032732069822455925 -> 0.03004188265707728
- link lb_shank: mass 0.043853773038341336 -> 0.12611282906621582
- link lb_thigh: mass 0.036696481476572916 -> 0.056003570757274454
- link lf_hip: mass 0.022572853506616163 -> 0.03004188265707728
- link lf_shank: mass 0.043853773038341336 -> 0.03565706349044272
- link lf_thigh: mass 0.036696481109002595 -> 0.056003570757274454
- link rb_hip: mass 0.032732069454885604 -> 0.03004188265707728
- link rb_shank: mass 0.043853773038341336 -> 0.12611282906621582
- link rb_thigh: mass 0.036696481109002595 -> 0.056003570757274454
- link rf_hip: mass 0.022568602179679133 -> 0.03004188265707728
- link rf_shank: mass 0.043853773038341336 -> 0.03565706349044272
- link rf_thigh: mass 0.036696481476572916 -> 0.056003570757274454
Joints:
- removed joint body,lb_hip_board
- removed joint body,lf_hip_board
- removed joint body,rb_hip_board
- removed joint body,rf_hip_board
- removed joint lb_hip,lb_thigh_motor
- removed joint lb_hip_board,lb_hip_motor
- removed joint lb_hip_motor,lb_hip
- removed joint lb_shank_board,lb_shank
- removed joint lb_shank_motor,lb_shank_board
- removed joint lb_thigh,lb_shank_motor
- removed joint lb_thigh_motor,lb_thigh
- removed joint lf_hip,lf_thigh_motor
- removed joint lf_hip_board,lf_hip_motor
- removed joint lf_hip_motor,lf_hip
- removed joint lf_shank_board,lf_shank
- removed joint lf_shank_motor,lf_shank_board
- removed joint lf_thigh,lf_shank_motor
- removed joint lf_thigh_motor,lf_thigh
- removed joint rb_hip,rb_thigh_motor
- removed joint rb_hip_board,rb_hip_motor
- removed joint rb_hip_motor,rb_hip
- removed joint rb_shank_board,rb_shank
- removed joint rb_shank_motor,rb_shank_board
- removed joint rb_thigh,rb_shank_motor
- removed joint rb_thigh_motor,rb_thigh
- removed joint rf_hip,rf_thigh_motor
- removed joint rf_hip_board,rf_hip_motor
- removed joint rf_hip_motor,rf_hip
- removed joint rf_shank_board,rf_shank
- removed joint rf_shank_motor,rf_shank_board
- removed joint rf_thigh,rf_shank_motor
- removed joint rf_thigh_motor,rf_thigh
- added joint body,lb_m1: type fixed, parent body, child lb_m1, origin xyz=0.013000000000000001 0.0 -0.17500000000000002 rpy=-1.5707963267948963 0.0 0.0, axis 1 0 0, limit effort=11 velocity=51
- added joint body,lf_m1: type fixed, parent body, child lf_m1, origin xyz=0.09 0.0 0.07 rpy=-1.5707963267948963 0.0 0.0, axis 1 0 0, limit effort=11 velocity=51
- added joint body,rb_m1: type fixed, parent body, child rb_m1, origin xyz=-0.013000000000000001 0.0 -0.17500000000000002 rpy=1.5707963267948963 2.220446049250313e-16 3.141592653589793, axis 1 0 0, limit effort=11 velocity=51
- added joint body,rf_m1: type fixed, parent body, child rf_m1, origin xyz=-0.09 0.0 0.07 rpy=1.5707963267948963 2.220446049250313e-16 3.141592653589793, axis 1 0 0, limit effort=11 velocity=51
- added joint lb_hip,lb_m2: type fixed, parent lb_hip, child lb_m2, origin xyz=0.051000000000000004 -0.0095 0.0 rpy=0.0 0.0 1.5707963267948963, axis 1 0 0, limit effort=11 velocity=51
- added joint lb_m1,lb_hip: type revolute, parent lb_m1, child lb_hip, origin xyz=0.032 0.0 0.0 rpy=0.0 0.0 0.0, axis 1 0 0, limit effort=11 velocity=51
- added joint lb_m2,lb_tc: type revolute, parent lb_m2, child lb_tc, origin xyz=0.032 0.0 0.0 rpy=0.0 0.0 0.0, axis 1 0 0, limit effort=11 velocity=51
- added joint lb_m3,lb_sc: type revolute, parent lb_m3, child lb_sc, origin xyz=0.032 0.0 0.0 rpy=0.0 0.0 0.0, axis 1 0 0, limit effort=11 velocity=51
- added joint lb_sc,lb_shank: type fixed, parent lb_sc, child lb_shank, origin xyz=-0.02 0.0 0.0 rpy=0.0 0.0 0.0, axis 1 0 0, limit effort=11 velocity=51
- added joint lb_tc,lb_thigh: type fixed, parent lb_tc, child lb_thigh, origin xyz=-0.021500000000000002 0.0 -0.145 rpy=0.0 0.0 1.5707963267948963, axis 1 0 0, limit effort=11 velocity=51
- added joint lb_thigh,lb_m3: type fixed, parent lb_thigh, child lb_m3, origin xyz=-0.012 0.0 0.0 rpy=0.0 0.0 0.0, axis 1 0 0, limit effort=11 velocity=51
- added joint lf_hip,lf_m2: type fixed, parent lf_hip, child lf_m2, origin xyz=0.051000000000000004 -0.0095 0.0 rpy=3.141592653589793 0.0 1.570796326794897, axis 1 0 0, limit effort=11 velocity=51
- added joint lf_m1,lf_hip: type revolute, parent lf_m1, child lf_hip, origin xyz=0.029 0.0 0.0 rpy=3.141592653589793 0.0 0.0, axis 1 0 0, limit effort=11 velocity=51
- added joint lf_m2,lf_tc: type revolute, parent lf_m2, child lf_tc, origin xyz=0.032 0.0 0.0 rpy=0.0 0.0 0.0, axis 1 0 0, limit effort=11 velocity=51
- added joint lf_m3,lf_sc: type revolute, parent lf_m3, child lf_sc, origin xyz=0.032 0.0 0.0 rpy=0.0 0.0 0.0, axis 1 0 0, limit effort=11 velocity=51
- added joint lf_sc,lf_shank: type fixed, parent lf_sc, child lf_shank, origin xyz=-0.02 0.0 -0.031 rpy=0.0 0.0 0.0, axis 1 0 0, limit effort=11 velocity=51
- added joint lf_tc,lf_thigh: type fixed, parent lf_tc, child lf_thigh, origin xyz=-0.021500000000000002 0.0 -0.145 rpy=0.0 0.0 -1.5707963267948963, axis 1 0 0, limit effort=11 velocity=51
- added joint lf_thigh,lf_m3: type fixed, parent lf_thigh, child lf_m3, origin xyz=-0.012 0.0 0.0 rpy=0.0 0.0 0.0, axis 1 0 0, limit effort=11 velocity=51
- added joint rb_hip,rb_m2: type fixed, parent rb_hip, child rb_m2, origin xyz=0.051000000000000004 -0.0095 0.0 rpy=3.141592653589793 0.0 1.570796326794897, axis 1 0 0, limit effort=11 velocity=51
- added joint rb_m1,rb_hip: type revolute, parent rb_m1, child rb_hip, origin xyz=0.032 0.0 0.0 rpy=3.141592653589793 0.0 0.0, axis 1 0 0, limit effort=11 velocity=51
- added joint rb_m2,rb_tc: type revolute, parent rb_m2, child rb_tc, origin xyz=0.032 0.0 0.0 rpy=0.0 0.0 0.0, axis 1 0 0, limit effort=11 velocity=51
- added joint rb_m3,rb_sc: type revolute, parent rb_m3, child rb_sc, origin xyz=0.032 0.0 0.0 rpy=0.0 0.0 0.0, axis 1 0 0, limit effort=11 velocity=51
- added joint rb_sc,rb_shank: type fixed, parent rb_sc, child rb_shank, origin xyz=-0.02 0.0 0.0 rpy=0.0 0.0 3.141592653589793, axis 1 0 0, limit effort=11 velocity=51
- added joint rb_tc,rb_thigh: type fixed, parent rb_tc, child rb_thigh, origin xyz=-0.021500000000000002 0.0 -0.145 rpy=0.0 0.0 -1.5707963267948963, axis 1 0 0, limit effort=11 velocity=51
- added joint rb_thigh,rb_m3: type fixed, parent rb_thigh, child rb_m3, origin xyz=-0.012 0.0 0.0 rpy=0.0 0.0 0.0, axis 1 0 0, limit effort=11 velocity=51
- added joint rf_hip,rf_m2: type fixed, parent rf_hip, child rf_m2, origin xyz=0.051000000000000004 -0.0095 0.0 rpy=0.0 0.0 1.5707963267948963, axis 1 0 0, limit effort=11 velocity=51
- added joint rf_m1,rf_hip: type revolute, parent rf_m1, child rf_hip, origin xyz=0.029 0.0 0.0 rpy=0.0 0.0 0.0, axis 1 0 0, limit effort=11 velocity=51
- added joint rf_m2,rf_tc: type revolute, parent rf_m2, child rf_tc, origin xyz=0.032 0.0 0.0 rpy=0.0 0.0 0.0, axis 1 0 0, limit effort=11 velocity=51
- added joint rf_m3,rf_sc: type revolute, parent rf_m3, child rf_sc, origin xyz=0.032 0.0 0.0 rpy=0.0 0.0 0.0, axis 1 0 0, limit effort=11 velocity=51
- added joint rf_sc,rf_shank: type fixed, parent rf_sc, child rf_shank, origin xyz=-0.02 0.0 -0.031 rpy=0.0 0.0 0.0, axis 1 0 0, limit effort=11 velocity=51
- added joint rf_tc,rf_thigh: type fixed, parent rf_tc, child rf_thigh, origin xyz=-0.021500000000000002 0.0 -0.145 rpy=0.0 0.0 1.5707963267948963, axis 1 0 0, limit effort=11 velocity=51
- added joint rf_thigh,rf_m3: type fixed, parent rf_thigh, child rf_m3, origin xyz=-0.012 0.0 0.0 rpy=0.0 0.0 0.0, axis 1 0 0, limit effort=11 velocity=51
